Commit message: change positioni of z1

File: low-level/resources/robots/b1z1/urdf/b2z1.urdf (robot description, URDF)
Before this commit: robot b2z1_description, 48 links, 47 joints
Joints:
- joint base_static_joint: origin xyz=0.3 0 0.09 rpy=0 0 0 -> xyz=0.1 0 0.09 rpy=0 0 0

Commit message: remove lidar

File: low-level/resources/robots/b1z1/urdf/b2z1.urdf (robot description, URDF)
Before this commit: robot b2z1_description, 48 links, 47 joints
Links:
- removed link lidar_link
Joints:
- removed joint joint_lidar
- joint base_static_joint: origin xyz=0.1 0 0.09 rpy=0 0 0 -> xyz=0.2 0 0.09 rpy=0 0 0

Commit message: b2z1_no_lidar

File: low-level/resources/robots/b1z1/urdf/b2z1.urdf (robot description, URDF)
Before this commit: robot b2z1_description, 48 links, 47 joints
Links:
- removed link lidar_link
Joints:
- removed joint joint_lidar
